File: hardware/uoo-light/single-board.sch (EAGLE design)
At the start: 27 parts

Commit message: second version of board. Mirrored elecromagnetic reeds, shorter pads in esp-12, better paths.added mount hole, bigger holes in my elements in library.
Parts:
- removed 3V1: 3V, pinhead:PINHD-1X1
- removed GND8: GND, pinhead:PINHD-1X1
- added C2, C3: (no value), rcl:CPOL-EUA/3216-18R
- added IC1: REG1117, burr-brown:REG1117
- added R10, R11, R7, R8, R9: (no value), rcl:R-EU_R0805
- added T1, T2: BC847, transistor:BC847
- C1: value (none) -> 100nF
- G: value (none) -> G
- IN: value (none) -> AC IN
- L: value (none) -> LOUT
- OUT: value (none) -> OUT
- S1: value (none) -> S1
- S2: value (none) -> S2
Connections:
- new net N$12: T2.C, U$2.-
- new net N$13: T1.C, U$3.-
- new net N$14: R7.2, R8.1, T2.B
- new net N$16: R10.1, R9.2, T1.B
- new net N$17: ESP-12.GPIO2, R11.1
- net +3V3: now also C3.+, IC1.VOUT, R11.2; no longer 3V1.1
- net GND: now also C2.-, C3.-, IC1.GND, R10.2, R8.2, T1.E, T2.E; no longer GND8.1, U$2.-, U$3.-
- net REL1: now also R7.1; no longer U$2.+
- net REL2: now also R9.1; no longer U$3.+
- net VCC: now also C2.+, IC1.VIN, U$2.+, U$3.+
Other:
- moved on the sheet: 3V, GND, L-2, R5, R6, RST
